File: Hardware/Escaneo2D/Escaneo2D.kicad_sch (KiCad schematic)
At the start: 7 parts, among them J1 OLED_I2C, J2 HC-SR04, J3 USB, J4 PWR, M1 Stepper_Motor_unipolar_5pin, U1 STM32-BlackPill, U2 ULN2003

Commit message: PCB Terminada
Parts:
- removed J4: PWR, TerminalBlock_Phoenix:TerminalBlock_Phoenix_MKDS-1,5-2-5.08_1x02_P5.08mm_Horizontal, symbol Connector:Screw_Terminal_01x02
- added H1, H2, H3, H4: MountingHole_Pad, MountingHole:MountingHole_2.2mm_M2_DIN965_Pad, symbol Mechanical:MountingHole_Pad
- added R1, R2, R3, R4: 10K, Resistor_THT:R_Axial_DIN0207_L6.3mm_D2.5mm_P7.62mm_Horizontal, symbol Device:R_Small
- added SW1, SW2, SW3, SW4: SW_Push, Button_Switch_THT:SW_PUSH-12mm, symbol Switch:SW_Push
Connections:
- net +3V3: now also R1.1, R2.1, R3.1, R4.1
- net BTN_DOWN: now also U1.35 (PB1), R2.2, SW2.2; no longer U1.33 (PA7)
- net BTN_ENTER: now also R3.2, SW3.2
- net BTN_RETURN: now also U1.33 (PA7), R4.2, SW4.2; no longer U1.35 (PB1)
- net BTN_UP: now also R1.2, SW1.2
- net GND: now also SW1.1, SW2.1, SW3.1, SW4.1
- no-connect marks 26 -> 30
Other:
- moved on the sheet: J1, J2, J3
